File: Hardware_Design_Files/Project_Bird_V2.1/Project_bird_V2.1.sch (EAGLE design)
At the start: 55 parts, among them U1 MS560702BA03-50, U10 MGSF2N02EL, U2 SST26VF032B-104I/SM, U3 LIS331DLHTR, U4 ZLDO1117G33TA, U5 MGSF2N02EL, U6 MGSF2N02EL, U7 MGSF2N02EL, U8 MGSF2N02EL, U9 ATMEGA32U4-AU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

Commit message: Created Flight Recorder Library to handle flight stats and flash recording.
Parts:
- J1, J2, J3, J4, J5, J6: device SparkFun-Connectors:CONN_022.54MM_SCREWTERM -> UTS_Rocketry_Main_EAGLE_Library:CONN_02-BACKUP2.54MM_SCREWTERM

Commit message: Reduced Program Size and Fixed Hardware 3D CAD
Parts:
- D1, D2: device SparkFun-DiscreteSemi:DIODE-SCHOTTKY-BAT20J -> UTS_Rocketry_Main_EAGLE_Library:DIODESOD-323F
- D3: device SparkFun-LED:LED3MM -> UTS_Rocketry_Main_EAGLE_Library:LED3MM-RED
- D4: device SparkFun-LED:LED3MM -> UTS_Rocketry_Main_EAGLE_Library:LED3MM-YELLOW
- ISP1: device adafruit:AVRISP-6 -> UTS_Rocketry_Main_EAGLE_Library:AVRISP-6
- J1, J2, J3, J4, J5, J6: device UTS_Rocketry_Main_EAGLE_Library:CONN_02-BACKUP2.54MM_SCREWTERM -> UTS_Rocketry_Main_EAGLE_Library:CONN_022.54MM_SCREWTERM
- S1: value MOMENTARY-SWITCH-SPST-PTH-6.0MM -> MOMENTARY-SWITCH-SPST; device SparkFun-Switches:MOMENTARY-SWITCH-SPST-PTH-6.0MM -> UTS_Rocketry_Main_EAGLE_Library:MOMENTARY-SWITCH-SPST
Changed lines of the file:
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@@
 <part name="U3" library="UTS_Rocketry_Main_EAGLE_Library" library_urn="urn:adsk.eagle:library:12961410" deviceset="LIS331DLHTR" device="" package3d_urn="urn:adsk.eagle:package:17632269/2"/>
 <part name="-X1" library="UTS_Rocketry_Main_EAGLE_Library" library_urn="urn:adsk.eagle:library:12961410" deviceset="PCB_USB_TYPE_A" device="" package3d_urn="urn:adsk.eagle:package:17078525/3"/>
-<part name="D1" library="SparkFun-DiscreteSemi" library_urn="urn:adsk.eagle:library:514" deviceset="DIODE-SCHOTTKY" device="-BAT20J" package3d_urn="urn:adsk.eagle:package:38441/1" value="1A"/>
-<part name="D2" library="SparkFun-DiscreteSemi" library_urn="urn:adsk.eagle:library:514" deviceset="DIODE-SCHOTTKY" device="-BAT20J" package3d_urn="urn:adsk.eagle:package:38441/1" value="1A"/>
+<part name="D1" library="UTS_Rocketry_Main_EAGLE_Library" library_urn="urn:adsk.eagle:library:12961410" deviceset="DIODE" device="SOD-323F" package3d_urn="urn:adsk.eagle:package:23083278/2" value="1A"/>
+<part name="D2" library="UTS_Rocketry_Main_EAGLE_Library" library_urn="urn:adsk.eagle:library:12961410" deviceset="DIODE" device="SOD-323F" package3d_urn="urn:adsk.eagle:package:23083278/2" value="1A"/>
 <part name="GND1" library="supply1" library_urn="urn:adsk.eagle:library:371" deviceset="GND" device=""/>
 <part name="GND2" library="supply1" library_urn="urn:adsk.eagle:library:371" deviceset="GND" device=""/>
@@
 <part name="R2" library="UTS_Rocketry_Main_EAGLE_Library" library_urn="urn:adsk.eagle:library:12961410" deviceset="RES_0805" device="" package3d_urn="urn:adsk.eagle:package:17632271/3" value="22R"/>
 <part name="U4" library="UTS_Rocketry_Main_EAGLE_Library" library_urn="urn:adsk.eagle:library:12961410" deviceset="ZLDO1117" device="G33TA" package3d_urn="urn:adsk.eagle:package:22594437/2"/>
-<part name="J1" library="UTS_Rocketry_Main_EAGLE_Library" library_urn="urn:adsk.eagle:library:12961410" deviceset="CONN_02-BACKUP" device="2.54MM_SCREWTERM" package3d_urn="urn:adsk.eagle:package:22823399/2"/>
-<part name="J2" library="UTS_Rocketry_Main_EAGLE_Library" library_urn="urn:adsk.eagle:library:12961410" deviceset="CONN_02-BACKUP" device="2.54MM_SCREWTERM" package3d_urn="urn:adsk.eagle:package:22823399/2"/>
-<part name="J3" library="UTS_Rocketry_Main_EAGLE_Library" library_urn="urn:adsk.eagle:library:12961410" deviceset="CONN_02-BACKUP" device="2.54MM_SCREWTERM" package3d_urn="urn:adsk.eagle:package:22823399/2"/>
-<part name="J4" library="UTS_Rocketry_Main_EAGLE_Library" library_urn="urn:adsk.eagle:library:12961410" deviceset="CONN_02-BACKUP" device="2.54MM_SCREWTERM" package3d_urn="urn:adsk.eagle:package:22823399/2"/>
-<part name="J5" library="UTS_Rocketry_Main_EAGLE_Library" library_urn="urn:adsk.eagle:library:12961410" deviceset="CONN_02-BACKUP" device="2.54MM_SCREWTERM" package3d_urn="urn:adsk.eagle:package:22823399/2"/>
+<part name="J1" library="UTS_Rocketry_Main_EAGLE_Library" library_urn="urn:adsk.eagle:library:12961410" deviceset="CONN_02" device="2.54MM_SCREWTERM" package3d_urn="urn:adsk.eagle:package:22823399/2"/>
+<part name="J2" library="UTS_Rocketry_Main_EAGLE_Library" library_urn="urn:adsk.eagle:library:12961410" deviceset="CONN_02" device="2.54MM_SCREWTERM" package3d_urn="urn:adsk.eagle:package:22823399/2"/>
+<part name="J3" library="UTS_Rocketry_Main_EAGLE_Library" library_urn="urn:adsk.eagle:library:12961410" deviceset="CONN_02" device="2.54MM_SCREWTERM" package3d_urn="urn:adsk.eagle:package:22823399/2"/>
+<part name="J4" library="UTS_Rocketry_Main_EAGLE_Library" library_urn="urn:adsk.eagle:library:12961410" deviceset="CONN_02" device="2.54MM_SCREWTERM" package3d_urn="urn:adsk.eagle:package:22823399/2"/>
+<part name="J5" library="UTS_Rocketry_Main_EAGLE_Library" library_urn="urn:adsk.eagle:library:12961410" deviceset="CONN_02" device="2.54MM_SCREWTERM" package3d_urn="urn:adsk.eagle:package:22823399/2"/>
 <part name="U5" library="UTS_Rocketry_Main_EAGLE_Library" library_urn="urn:adsk.eagle:library:12961410" deviceset="MGSF2N02EL" device="" package3d_urn="urn:adsk.eagle:package:22297200/2"/>
 <part name="P+1" library="supply1" library_urn="urn:adsk.eagle:library:371" deviceset="+12V" device=""/>
@@
 <part name="R14" library="UTS_Rocketry_Main_EAGLE_Library" library_urn="urn:adsk.eagle:library:12961410" deviceset="RES_0805" device="" package3d_urn="urn:adsk.eagle:package:17632271/3" value="33K"/>
 <part name="GND6" library="supply1" library_urn="urn:adsk.eagle:library:371" deviceset="GND" device=""/>
-<part name="J6" library="UTS_Rocketry_Main_EAGLE_Library" library_urn="urn:adsk.eagle:library:12961410" deviceset="CONN_02-BACKUP" device="2.54MM_SCREWTERM" package3d_urn="urn:adsk.eagle:package:22823399/2"/>
+<part name="J6" library="UTS_Rocketry_Main_EAGLE_Library" library_urn="urn:adsk.eagle:library:12961410" deviceset="CONN_02" device="2.54MM_SCREWTERM" package3d_urn="urn:adsk.eagle:package:22823399/2"/>
 <part name="GND7" library="supply1" library_urn="urn:adsk.eagle:library:371" deviceset="GND" device=""/>
 <part name="U$2" library="UTS_Rocketry_Main_EAGLE_Library" library_urn="urn:adsk.eagle:library:12961410" deviceset="TITLE_BLOCK_PAGE_TEMPLATE_A4" device="">
@@
 </part>
 <part name="U9" library="UTS_Rocketry_Main_EAGLE_Library" library_urn="urn:adsk.eagle:library:12961410" deviceset="ATMEGA32U4-AU" device="" package3d_urn="urn:adsk.eagle:package:22596034/2"/>
-<part name="Y1" library="UTS_Rocketry_Main_EAGLE_Library" library_urn="urn:adsk.eagle:library:12961410" deviceset="RESONATOR-CSTCE" device="8M00G55-R0" package3d_urn="urn:adsk.eagle:package:37551/1" value="8MHz"/>
+<part name="Y1" library="UTS_Rocketry_Main_EAGLE_Library" library_urn="urn:adsk.eagle:library:12961410" deviceset="RESONATOR-CSTCE" device="8M00G55-R0" package3d_urn="urn:adsk.eagle:package:23083263/2" value="8MHz"/>
 <part name="GND8" library="supply1" library_urn="urn:adsk.eagle:library:371" deviceset="GND" device=""/>
 <part name="C3" library="UTS_Rocketry_Main_EAGLE_Library" library_urn="urn:adsk.eagle:library:12961410" deviceset="CAP_0805" device="" package3d_urn="urn:adsk.eagle:package:17632272/3" value="0.1uF"/>
@@
 <part name="+3V10" library="supply1" library_urn="urn:adsk.eagle:library:371" deviceset="+3V3" device=""/>
 <part name="+3V11" library="supply1" library_urn="urn:adsk.eagle:library:371" deviceset="+3V3" device=""/>
-<part name="ISP1" library="adafruit" library_urn="urn:adsk.eagle:library:420" deviceset="AVRISP" device="-6" package3d_urn="urn:adsk.eagle:package:6240744/1"/>
+<part name="ISP1" library="UTS_Rocketry_Main_EAGLE_Library" library_urn="urn:adsk.eagle:library:12961410" deviceset="AVRISP" device="-6" package3d_urn="urn:adsk.eagle:package:23083285/2"/>
 <part name="GND18" library="supply1" library_urn="urn:adsk.eagle:library:371" deviceset="GND" device=""/>
-<part name="S1" library="SparkFun-Switches" library_urn="urn:adsk.eagle:library:535" deviceset="MOMENTARY-SWITCH-SPST" device="-PTH-6.0MM" package3d_urn="urn:adsk.eagle:package:40163/1"/>
+<part name="S1" library="UTS_Rocketry_Main_EAGLE_Library" library_urn="urn:adsk.eagle:library:12961410" deviceset="MOMENTARY-SWITCH-SPST" device="" package3d_urn="urn:adsk.eagle:package:23083248/2"/>
 <part name="GND19" library="supply1" library_urn="urn:adsk.eagle:library:371" deviceset="GND" device=""/>
-<part name="D3" library="SparkFun-LED" library_urn="urn:adsk.eagle:library:529" deviceset="LED" device="3MM" package3d_urn="urn:adsk.eagle:package:39361/1"/>
-<part name="D4" library="SparkFun-LED" library_urn="urn:adsk.eagle:library:529" deviceset="LED" device="3MM" package3d_urn="urn:adsk.eagle:package:39361/1"/>
+<part name="D3" library="UTS_Rocketry_Main_EAGLE_Library" library_urn="urn:adsk.eagle:library:12961410" deviceset="LED3MM" device="-RED" package3d_urn="urn:adsk.eagle:package:23083266/2"/>
+<part name="D4" library="UTS_Rocketry_Main_EAGLE_Library" library_urn="urn:adsk.eagle:library:12961410" deviceset="LED3MM" device="-YELLOW" package3d_urn="urn:adsk.eagle:package:23083266/2"/>
 <part name="R17" library="UTS_Rocketry_Main_EAGLE_Library" library_urn="urn:adsk.eagle:library:12961410" deviceset="RES_0805" device="" package3d_urn="urn:adsk.eagle:package:17632271/3" value="330R"/>
 <part name="R20" library="UTS_Rocketry_Main_EAGLE_Library" library_urn="urn:adsk.eagle:library:12961410" deviceset="RES_0805" device="" package3d_urn="urn:adsk.eagle:package:17632271/3" value="330R"/>
@@
 <part name="GND22" library="supply1" library_urn="urn:adsk.eagle:library:371" deviceset="GND" device=""/>
 <part name="R21" library="UTS_Rocketry_Main_EAGLE_Library" library_urn="urn:adsk.eagle:library:12961410" deviceset="RES_0805" device="" package3d_urn="urn:adsk.eagle:package:17632271/3" value="330R"/>
-<part name="LS1" library="UTS_Rocketry_Main_EAGLE_Library" library_urn="urn:adsk.eagle:library:12961410" deviceset="BUZZER" device="-SMD" package3d_urn="urn:adsk.eagle:package:38552/1"/>
+<part name="LS1" library="UTS_Rocketry_Main_EAGLE_Library" library_urn="urn:adsk.eagle:library:12961410" deviceset="BUZZER" device="-SMD" package3d_urn="urn:adsk.eagle:package:23083286/2"/>
 </parts>
 <sheets>
@@
 <instance part="D1" gate="G$1" x="73.66" y="175.26" smashed="yes">
 <attribute name="NAME" x="71.12" y="177.292" size="1.778" layer="95" font="vector"/>
-<attribute name="VALUE" x="71.12" y="173.228" size="1.778" layer="96" font="vector" align="top-left"/>
 </instance>
 <instance part="D2" gate="G$1" x="73.66" y="144.78" smashed="yes">
 <attribute name="NAME" x="71.12" y="146.812" size="1.778" layer="95" font="vector"/>
-<attribute name="VALUE" x="71.12" y="142.748" size="1.778" layer="96" font="vector" align="top-left"/>
 </instance>
 <instance part="GND1" gate="1" x="33.02" y="157.48" smashed="yes">
